Commit message: Rename (#62)
* renamed dynaarm_driver -> duatic_dynaarm_driver

File: urdf/common/baracuda12/dynaarm_parameters.urdf.xacro (robot description, xacro)
@@ -1,4 +1,5 @@
+<?xml version="1.0"?>
 <!--
-Copyright 2024 Duatic AG
+Copyright 2026 Duatic AG
 Redistribution and use in source and binary forms, with or without modification, are permitted
 provided that the following conditions are met:
@@ -340,5 +341,5 @@
         <geometry>
           <mesh
-            filename="file://$(find dynaarm_description)/meshes/baracuda12/collision_meshes/base_collision_mesh.stl"
+            filename="file://$(find duatic_dynaarm_description)/meshes/baracuda12/collision_meshes/base_collision_mesh.stl"
             scale="1 1 1" />
         </geometry>
@@ -350,5 +351,5 @@
         <geometry>
           <mesh
-            filename="file://$(find dynaarm_description)/meshes/baracuda12/collision_meshes/shoulder_collision_mesh.stl"
+            filename="file://$(find duatic_dynaarm_description)/meshes/baracuda12/collision_meshes/shoulder_collision_mesh.stl"
             scale="1 1 1" />
         </geometry>
@@ -360,5 +361,5 @@
         <geometry>
           <mesh
-            filename="file://$(find dynaarm_description)/meshes/baracuda12/collision_meshes/upperarm_collision_mesh.stl"
+            filename="file://$(find duatic_dynaarm_description)/meshes/baracuda12/collision_meshes/upperarm_collision_mesh.stl"
             scale="1 1 1" />
         </geometry>
@@ -370,5 +371,5 @@
         <geometry>
           <mesh
-            filename="file://$(find dynaarm_description)/meshes/baracuda12/collision_meshes/elbow_collision_mesh.stl"
+            filename="file://$(find duatic_dynaarm_description)/meshes/baracuda12/collision_meshes/elbow_collision_mesh.stl"
             scale="1 1 1" />
         </geometry>
@@ -380,5 +381,5 @@
         <geometry>
           <mesh
-            filename="file://$(find dynaarm_description)/meshes/baracuda12/collision_meshes/forearm_collision_mesh.stl"
+            filename="file://$(find duatic_dynaarm_description)/meshes/baracuda12/collision_meshes/forearm_collision_mesh.stl"
             scale="1 1 1" />
         </geometry>
@@ -390,5 +391,5 @@
         <geometry>
           <mesh
-            filename="file://$(find dynaarm_description)/meshes/baracuda12/collision_meshes/wrist1_collision_mesh.stl"
+            filename="file://$(find duatic_dynaarm_description)/meshes/baracuda12/collision_meshes/wrist1_collision_mesh.stl"
             scale="1 1 1" />
         </geometry>
@@ -400,5 +401,5 @@
         <geometry>
           <mesh
-            filename="file://$(find dynaarm_description)/meshes/baracuda12/collision_meshes/wrist2_collision_mesh.stl"
+            filename="file://$(find duatic_dynaarm_description)/meshes/baracuda12/collision_meshes/wrist2_collision_mesh.stl"
             scale="1 1 1" />
         </geometry>

File: urdf/common/dynaarm.ros2control.xacro (robot description, xacro)
@@ -1,10 +1,23 @@
 <?xml version="1.0"?>
 <!--
-Copyright 2024 Duatic AG
-Redistribution and use in source and binary forms, with or without modification, are permitted provided that the following conditions are met:
-1. Redistributions of source code must retain the above copyright notice, this list of conditions and the following disclaimer.
-2. Redistributions in binary form must reproduce the above copyright notice, this list of conditions and the following disclaimer in the documentation and/or other materials provided with the distribution.
-3. Neither the name of the copyright holder nor the names of its contributors may be used to endorse or promote products derived from this software without specific prior written permission.
-THIS SOFTWARE IS PROVIDED BY THE COPYRIGHT HOLDERS AND CONTRIBUTORS “AS IS” AND ANY EXPRESS OR IMPLIED WARRANTIES, INCLUDING, BUT NOT LIMITED TO, THE IMPLIED WARRANTIES OF MERCHANTABILITY AND FITNESS FOR A PARTICULAR PURPOSE ARE DISCLAIMED. IN NO EVENT SHALL THE COPYRIGHT HOLDER OR CONTRIBUTORS BE LIABLE FOR ANY DIRECT, INDIRECT, INCIDENTAL, SPECIAL, EXEMPLARY, OR CONSEQUENTIAL DAMAGES (INCLUDING, BUT NOT LIMITED TO, PROCUREMENT OF SUBSTITUTE GOODS OR SERVICES; LOSS OF USE, DATA, OR PROFITS; OR BUSINESS INTERRUPTION) HOWEVER CAUSED AND ON ANY THEORY OF LIABILITY, WHETHER IN CONTRACT, STRICT LIABILITY, OR TORT (INCLUDING NEGLIGENCE OR OTHERWISE) ARISING IN ANY WAY OUT OF THE USE OF THIS SOFTWARE, EVEN IF ADVISED OF THE POSSIBILITY OF SUCH DAMAGE.
+Copyright 2026 Duatic AG
+Redistribution and use in source and binary forms, with or without modification, are permitted
+provided that the following conditions are met:
+1. Redistributions of source code must retain the above copyright notice, this list of conditions
+and the following disclaimer.
+2. Redistributions in binary form must reproduce the above copyright notice, this list of
+conditions and the following disclaimer in the documentation and/or other materials provided with
+the distribution.
+3. Neither the name of the copyright holder nor the names of its contributors may be used to
+endorse or promote products derived from this software without specific prior written permission.
+THIS SOFTWARE IS PROVIDED BY THE COPYRIGHT HOLDERS AND CONTRIBUTORS “AS IS” AND ANY EXPRESS OR
+IMPLIED WARRANTIES, INCLUDING, BUT NOT LIMITED TO, THE IMPLIED WARRANTIES OF MERCHANTABILITY AND
+FITNESS FOR A PARTICULAR PURPOSE ARE DISCLAIMED. IN NO EVENT SHALL THE COPYRIGHT HOLDER OR
+CONTRIBUTORS BE LIABLE FOR ANY DIRECT, INDIRECT, INCIDENTAL, SPECIAL, EXEMPLARY, OR CONSEQUENTIAL
+DAMAGES (INCLUDING, BUT NOT LIMITED TO, PROCUREMENT OF SUBSTITUTE GOODS OR SERVICES; LOSS OF USE,
+DATA, OR PROFITS; OR BUSINESS INTERRUPTION) HOWEVER CAUSED AND ON ANY THEORY OF LIABILITY, WHETHER
+IN CONTRACT, STRICT LIABILITY, OR TORT (INCLUDING NEGLIGENCE OR OTHERWISE) ARISING IN ANY WAY OUT
+OF
+THE USE OF THIS SOFTWARE, EVEN IF ADVISED OF THE POSSIBILITY OF SUCH DAMAGE.
 -->
 <robot xmlns:xacro="http://www.ros.org/wiki/xacro">
@@ -63,5 +76,5 @@
         </xacro:if>
         <xacro:if value="${mode == 'mock'}">
-          <plugin>dynaarm_driver/DynaarmMockHardwareInterface</plugin>
+          <plugin>duatic_dynaarm_driver/DynaarmMockHardwareInterface</plugin>
           <param name="tf_prefix">${tf_prefix}</param>
           <param name="start_in_freeze_mode">${start_in_freeze_mode}</param>
@@ -71,5 +84,5 @@
         </xacro:if>
         <xacro:if value="${mode == 'real'}">
-          <plugin>dynaarm_driver/DynaArmHardwareInterface</plugin>
+          <plugin>duatic_dynaarm_driver/DynaArmHardwareInterface</plugin>
           <param name="ethercat_bus">${ethercat_bus}</param>
           <param name="tf_prefix">${tf_prefix}</param>

File: urdf/common/dynaarm_common.urdf.xacro (robot description, xacro)
@@ -1,5 +1,5 @@
 <?xml version="1.0"?>
 <!--
-Copyright 2024 Duatic AG
+Copyright 2026 Duatic AG
 Redistribution and use in source and binary forms, with or without modification, are permitted
 provided that the following conditions are met:
@@ -31,5 +31,5 @@
                 <geometry>
                     <mesh
-                        filename="file://$(find dynaarm_description)/meshes/${version}/${file_name}"
+                        filename="file://$(find duatic_dynaarm_description)/meshes/${version}/${file_name}"
                         scale="1.0 1.0 1.0" />
                 </geometry>
@@ -51,5 +51,5 @@
                 <geometry>
                     <mesh
-                        filename="file://$(find dynaarm_description)/meshes/${version}/${file_name}"
+                        filename="file://$(find duatic_dynaarm_description)/meshes/${version}/${file_name}"
                         scale="1.0 1.0 1.0" />
                 </geometry>
@@ -67,5 +67,5 @@
                 <geometry>
                     <mesh
-                        filename="file://$(find dynaarm_description)/meshes/${version}/${file_name}"
+                        filename="file://$(find duatic_dynaarm_description)/meshes/${version}/${file_name}"
                         scale="1.0 1.0 1.0" />
                 </geometry>

File: urdf/dynaarm.urdf.xacro (robot description, xacro)
@@ -1,5 +1,5 @@
 <?xml version="1.0"?>
 <!--
-Copyright 2025 Duatic AG
+Copyright 2026 Duatic AG
 Redistribution and use in source and binary forms, with or without modification, are permitted
 provided that the following conditions are met:
@@ -28,10 +28,10 @@
     params="tf_prefix parent_link collision:='simple' dof mode ethercat_bus drive_order:='' start_in_freeze_mode:=false drive_parameter_folder:='' covers version *origin">
     <!-- Allow the user to pass the drive order file -->
-    <xacro:property name="default_drive_order_file" value="$(find dynaarm_description)/urdf/common/${version}/drive_order.yaml" />
+    <xacro:property name="default_drive_order_file" value="$(find duatic_dynaarm_description)/urdf/common/${version}/drive_order.yaml" />
     <xacro:property name="drive_order_file" value="${default_drive_order_file if drive_order == '' else drive_order}" />
     <!-- Obtain the EtherCAT drive order (address order list) -->
     <xacro:property name="ethercat_addresses" value="${xacro.load_yaml(drive_order_file)}"/>
     <!--Allow the user to pass a custom folder for drive parameters-->
-    <xacro:property name="default_drive_parameter_folder" value="$(find dynaarm_driver)/config/${version}" />
+    <xacro:property name="default_drive_parameter_folder" value="$(find duatic_dynaarm_driver)/config/${version}" />
     <xacro:if value="${drive_parameter_folder == ''}">
       <xacro:property name="drive_parameter_folder_internal" value="${default_drive_parameter_folder}" />
@@ -42,8 +42,8 @@
     <!-- Set ee_parent based on the specified DoF -->
     <xacro:property name="ee_parent" value="${base}" />
-    <xacro:include filename="$(find dynaarm_description)/urdf/common/dynaarm_common.urdf.xacro" />
+    <xacro:include filename="$(find duatic_dynaarm_description)/urdf/common/dynaarm_common.urdf.xacro" />
     <!-- Include the version specific information and also load the ethercat addresses from the drive file -->
-    <xacro:include filename="$(find dynaarm_description)/urdf/common/${version}/dynaarm_parameters.urdf.xacro" />
-    <xacro:include filename="$(find dynaarm_description)/urdf/common/dynaarm.ros2control.xacro" />
+    <xacro:include filename="$(find duatic_dynaarm_description)/urdf/common/${version}/dynaarm_parameters.urdf.xacro" />
+    <xacro:include filename="$(find duatic_dynaarm_description)/urdf/common/dynaarm.ros2control.xacro" />
     <xacro:dynaarm_joint_fixed joint_name="${joint_base_name}"
       parent="${parent_link}"

File: urdf/dynaarm_standalone.urdf.xacro (robot description, xacro)
@@ -1,9 +1,23 @@
+<?xml version="1.0"?>
 <!--
-Copyright 2024 Duatic AG
-Redistribution and use in source and binary forms, with or without modification, are permitted provided that the following conditions are met:
-1. Redistributions of source code must retain the above copyright notice, this list of conditions and the following disclaimer.
-2. Redistributions in binary form must reproduce the above copyright notice, this list of conditions and the following disclaimer in the documentation and/or other materials provided with the distribution.
-3. Neither the name of the copyright holder nor the names of its contributors may be used to endorse or promote products derived from this software without specific prior written permission.
-THIS SOFTWARE IS PROVIDED BY THE COPYRIGHT HOLDERS AND CONTRIBUTORS “AS IS” AND ANY EXPRESS OR IMPLIED WARRANTIES, INCLUDING, BUT NOT LIMITED TO, THE IMPLIED WARRANTIES OF MERCHANTABILITY AND FITNESS FOR A PARTICULAR PURPOSE ARE DISCLAIMED. IN NO EVENT SHALL THE COPYRIGHT HOLDER OR CONTRIBUTORS BE LIABLE FOR ANY DIRECT, INDIRECT, INCIDENTAL, SPECIAL, EXEMPLARY, OR CONSEQUENTIAL DAMAGES (INCLUDING, BUT NOT LIMITED TO, PROCUREMENT OF SUBSTITUTE GOODS OR SERVICES; LOSS OF USE, DATA, OR PROFITS; OR BUSINESS INTERRUPTION) HOWEVER CAUSED AND ON ANY THEORY OF LIABILITY, WHETHER IN CONTRACT, STRICT LIABILITY, OR TORT (INCLUDING NEGLIGENCE OR OTHERWISE) ARISING IN ANY WAY OUT OF THE USE OF THIS SOFTWARE, EVEN IF ADVISED OF THE POSSIBILITY OF SUCH DAMAGE.
+Copyright 2026 Duatic AG
+Redistribution and use in source and binary forms, with or without modification, are permitted
+provided that the following conditions are met:
+1. Redistributions of source code must retain the above copyright notice, this list of conditions
+and the following disclaimer.
+2. Redistributions in binary form must reproduce the above copyright notice, this list of
+conditions and the following disclaimer in the documentation and/or other materials provided with
+the distribution.
+3. Neither the name of the copyright holder nor the names of its contributors may be used to
+endorse or promote products derived from this software without specific prior written permission.
+THIS SOFTWARE IS PROVIDED BY THE COPYRIGHT HOLDERS AND CONTRIBUTORS “AS IS” AND ANY EXPRESS OR
+IMPLIED WARRANTIES, INCLUDING, BUT NOT LIMITED TO, THE IMPLIED WARRANTIES OF MERCHANTABILITY AND
+FITNESS FOR A PARTICULAR PURPOSE ARE DISCLAIMED. IN NO EVENT SHALL THE COPYRIGHT HOLDER OR
+CONTRIBUTORS BE LIABLE FOR ANY DIRECT, INDIRECT, INCIDENTAL, SPECIAL, EXEMPLARY, OR CONSEQUENTIAL
+DAMAGES (INCLUDING, BUT NOT LIMITED TO, PROCUREMENT OF SUBSTITUTE GOODS OR SERVICES; LOSS OF USE,
+DATA, OR PROFITS; OR BUSINESS INTERRUPTION) HOWEVER CAUSED AND ON ANY THEORY OF LIABILITY, WHETHER
+IN CONTRACT, STRICT LIABILITY, OR TORT (INCLUDING NEGLIGENCE OR OTHERWISE) ARISING IN ANY WAY OUT
+OF
+THE USE OF THIS SOFTWARE, EVEN IF ADVISED OF THE POSSIBILITY OF SUCH DAMAGE.
 -->
 <robot name="dynaarm" xmlns:xacro="http://www.ros.org/wiki/xacro">
@@ -25,6 +39,5 @@
   <!-- Path to ros2_control controller config file -->
   <xacro:arg name="controller_path" default="" />
-  <xacro:arg name="namespace" default="" />
-  <xacro:include filename="$(find dynaarm_description)/urdf/dynaarm.urdf.xacro" />
+  <xacro:include filename="$(find duatic_dynaarm_description)/urdf/dynaarm.urdf.xacro" />
   <link name="base_link" />
   <!-- create an instance of the dynaarm xacro macro and fix its base, move it up such that it doesn't intersect with the ground -->

File: urdf/dynaarm_standalone_dual.urdf.xacro (robot description, xacro)
@@ -1,9 +1,23 @@
+<?xml version="1.0"?>
 <!--
-Copyright 2024 Duatic AG
-Redistribution and use in source and binary forms, with or without modification, are permitted provided that the following conditions are met:
-1. Redistributions of source code must retain the above copyright notice, this list of conditions and the following disclaimer.
-2. Redistributions in binary form must reproduce the above copyright notice, this list of conditions and the following disclaimer in the documentation and/or other materials provided with the distribution.
-3. Neither the name of the copyright holder nor the names of its contributors may be used to endorse or promote products derived from this software without specific prior written permission.
-THIS SOFTWARE IS PROVIDED BY THE COPYRIGHT HOLDERS AND CONTRIBUTORS “AS IS” AND ANY EXPRESS OR IMPLIED WARRANTIES, INCLUDING, BUT NOT LIMITED TO, THE IMPLIED WARRANTIES OF MERCHANTABILITY AND FITNESS FOR A PARTICULAR PURPOSE ARE DISCLAIMED. IN NO EVENT SHALL THE COPYRIGHT HOLDER OR CONTRIBUTORS BE LIABLE FOR ANY DIRECT, INDIRECT, INCIDENTAL, SPECIAL, EXEMPLARY, OR CONSEQUENTIAL DAMAGES (INCLUDING, BUT NOT LIMITED TO, PROCUREMENT OF SUBSTITUTE GOODS OR SERVICES; LOSS OF USE, DATA, OR PROFITS; OR BUSINESS INTERRUPTION) HOWEVER CAUSED AND ON ANY THEORY OF LIABILITY, WHETHER IN CONTRACT, STRICT LIABILITY, OR TORT (INCLUDING NEGLIGENCE OR OTHERWISE) ARISING IN ANY WAY OUT OF THE USE OF THIS SOFTWARE, EVEN IF ADVISED OF THE POSSIBILITY OF SUCH DAMAGE.
+Copyright 2026 Duatic AG
+Redistribution and use in source and binary forms, with or without modification, are permitted
+provided that the following conditions are met:
+1. Redistributions of source code must retain the above copyright notice, this list of conditions
+and the following disclaimer.
+2. Redistributions in binary form must reproduce the above copyright notice, this list of
+conditions and the following disclaimer in the documentation and/or other materials provided with
+the distribution.
+3. Neither the name of the copyright holder nor the names of its contributors may be used to
+endorse or promote products derived from this software without specific prior written permission.
+THIS SOFTWARE IS PROVIDED BY THE COPYRIGHT HOLDERS AND CONTRIBUTORS “AS IS” AND ANY EXPRESS OR
+IMPLIED WARRANTIES, INCLUDING, BUT NOT LIMITED TO, THE IMPLIED WARRANTIES OF MERCHANTABILITY AND
+FITNESS FOR A PARTICULAR PURPOSE ARE DISCLAIMED. IN NO EVENT SHALL THE COPYRIGHT HOLDER OR
+CONTRIBUTORS BE LIABLE FOR ANY DIRECT, INDIRECT, INCIDENTAL, SPECIAL, EXEMPLARY, OR CONSEQUENTIAL
+DAMAGES (INCLUDING, BUT NOT LIMITED TO, PROCUREMENT OF SUBSTITUTE GOODS OR SERVICES; LOSS OF USE,
+DATA, OR PROFITS; OR BUSINESS INTERRUPTION) HOWEVER CAUSED AND ON ANY THEORY OF LIABILITY, WHETHER
+IN CONTRACT, STRICT LIABILITY, OR TORT (INCLUDING NEGLIGENCE OR OTHERWISE) ARISING IN ANY WAY OUT
+OF
+THE USE OF THIS SOFTWARE, EVEN IF ADVISED OF THE POSSIBILITY OF SUCH DAMAGE.
 -->
 <robot name="dynaarm" xmlns:xacro="http://www.ros.org/wiki/xacro">
@@ -24,5 +38,5 @@
   <!-- Path to ros2_control controller config file -->
   <xacro:arg name="controller_path" default="" />
-  <xacro:include filename="$(find dynaarm_description)/urdf/dynaarm.urdf.xacro" />
+  <xacro:include filename="$(find duatic_dynaarm_description)/urdf/dynaarm.urdf.xacro" />
   <link name="base_link" />
   <!-- create two dynaarms and fix their bases, move them up such that they do not intersect with the ground -->
@@ -50,5 +64,5 @@
   <!-- DynaArm Gazebo Ros2 Control-->
   <!-- Gazebo Ros2 Control -->
-  <xacro:include filename="$(find duatic_control)/urdf/plugins.urdf.xacro" />
+  <xacro:include filename="$(find duatic_duatic_control)/urdf/plugins.urdf.xacro" />
   <xacro:control namespace="$(arg namespace)">
     <remapping>cmd_vel:=cmd_vel</remapping> <!-- TODO: This line only exists, because otherwise the xacro doesn't compile -->
