Commit message: added namespace

File: urdf/common/dynaarm.ros2control.xacro (robot description, xacro)
@@ -49,11 +49,11 @@
     </joint>
   </xacro:macro>
-  <xacro:macro name="dynaarm_ros2_control" params="tf_prefix ethercat_bus start_in_freeze_mode drive_parameter_folder drive_parameter_folder_default ethercat_addresses mode">
+  <xacro:macro name="dynaarm_ros2_control" params="tf_prefix namespace:='' ethercat_bus start_in_freeze_mode drive_parameter_folder drive_parameter_folder_default ethercat_addresses mode">
     <ros2_control name="${tf_prefix}DynaarmSystem" type="system">
       <hardware>
         <xacro:if value="${mode == 'isaac'}">
           <plugin>joint_state_topic_hardware_interface/JointStateTopicSystem</plugin>
-          <param name="joint_states_topic">/isaac_joint_states</param>
-          <param name="joint_commands_topic">/isaac_joint_command</param>
+          <param name="joint_states_topic">${namespace}/isaac_joint_states</param>
+          <param name="joint_commands_topic">${namespace}/${tf_prefix}isaac_joint_command</param>
           <!-- Isaac wraps joint angles, this helps un-wrap them -->
           <param name="sum_wrapped_joint_states">true</param>

Commit message: Feature/isaac sim (#58)
* Added setup for isaac-sim

* added namespace

* pleased pre-commit

* Removed default namespace

File: urdf/common/dynaarm.ros2control.xacro (robot description, xacro)
@@ -31,13 +31,32 @@
     <command_interface name="d_gain" />
   </xacro:macro>
-  <xacro:macro name="dynaarm_ros2control_joint" params="name address">
+  <xacro:macro name="dynaarm_ros2control_joint" params="name address mode">
     <joint name="${name}">
-      <param name="address">${address}</param>
-      <xacro:dynaarm_joint_ros2control_joint_interfaces />
+      <xacro:if value="${mode != 'isaac'}">
+        <param name="address">${address}</param>
+        <xacro:dynaarm_joint_ros2control_joint_interfaces />
+      </xacro:if>
+      <xacro:if value="${mode == 'isaac'}">
+        <command_interface name="position" />
+        <command_interface name="velocity" />
+        <command_interface name="effort" />
+        <state_interface name="position">
+          <param name="initial_value">0.0</param>
+        </state_interface>
+        <state_interface name="velocity" />
+        <state_interface name="effort" />
+      </xacro:if>
     </joint>
   </xacro:macro>
-  <xacro:macro name="dynaarm_ros2_control" params="tf_prefix ethercat_bus start_in_freeze_mode drive_parameter_folder drive_parameter_folder_default ethercat_addresses">
+  <xacro:macro name="dynaarm_ros2_control" params="tf_prefix namespace:='' ethercat_bus start_in_freeze_mode drive_parameter_folder drive_parameter_folder_default ethercat_addresses mode">
     <ros2_control name="${tf_prefix}DynaarmSystem" type="system">
       <hardware>
+        <xacro:if value="${mode == 'isaac'}">
+          <plugin>joint_state_topic_hardware_interface/JointStateTopicSystem</plugin>
+          <param name="joint_states_topic">${namespace}/isaac_joint_states</param>
+          <param name="joint_commands_topic">${namespace}/${tf_prefix}isaac_joint_command</param>
+          <!-- Isaac wraps joint angles, this helps un-wrap them -->
+          <param name="sum_wrapped_joint_states">true</param>
+        </xacro:if>
         <xacro:if value="${mode == 'sim'}">
           <plugin>gz_ros2_control/GazeboSimSystem</plugin>
@@ -61,24 +80,26 @@
       </hardware>
       <xacro:if value="${dof >= 1}">
-        <xacro:dynaarm_ros2control_joint name="${tf_prefix}shoulder_rotation" address="${ethercat_addresses['shoulder_rotation']}" />
+        <xacro:dynaarm_ros2control_joint name="${tf_prefix}shoulder_rotation" address="${ethercat_addresses['shoulder_rotation']}" mode="${mode}" />
       </xacro:if>
       <xacro:if value="${dof >= 2}">
-        <xacro:dynaarm_ros2control_joint name="${tf_prefix}shoulder_flexion" address="${ethercat_addresses['shoulder_flexion']}" />
+        <xacro:dynaarm_ros2control_joint name="${tf_prefix}shoulder_flexion" address="${ethercat_addresses['shoulder_flexion']}" mode="${mode}" />
       </xacro:if>
       <xacro:if value="${dof >= 3}">
-        <xacro:dynaarm_ros2control_joint name="${tf_prefix}elbow_flexion" address="${ethercat_addresses['elbow_flexion']}" />
+        <xacro:dynaarm_ros2control_joint name="${tf_prefix}elbow_flexion" address="${ethercat_addresses['elbow_flexion']}" mode="${mode}" />
       </xacro:if>
       <xacro:if value="${dof >= 4}">
-        <xacro:dynaarm_ros2control_joint name="${tf_prefix}forearm_rotation" address="${ethercat_addresses['forearm_rotation']}" />
+        <xacro:dynaarm_ros2control_joint name="${tf_prefix}forearm_rotation" address="${ethercat_addresses['forearm_rotation']}" mode="${mode}" />
       </xacro:if>
       <xacro:if value="${dof >= 5}">
-        <xacro:dynaarm_ros2control_joint name="${tf_prefix}wrist_flexion" address="${ethercat_addresses['wrist_flexion']}" />
+        <xacro:dynaarm_ros2control_joint name="${tf_prefix}wrist_flexion" address="${ethercat_addresses['wrist_flexion']}" mode="${mode}" />
       </xacro:if>
       <xacro:if value="${dof >= 6}">
-        <xacro:dynaarm_ros2control_joint name="${tf_prefix}wrist_rotation" address="${ethercat_addresses['wrist_rotation']}" />
+        <xacro:dynaarm_ros2control_joint name="${tf_prefix}wrist_rotation" address="${ethercat_addresses['wrist_rotation']}" mode="${mode}" />
       </xacro:if>
-      <gpio name="${tf_prefix}DynaarmSystem">
-       <command_interface name="freeze_mode" />
-      </gpio>
+      <xacro:if value="${mode != 'isaac'}">
+        <gpio name="${tf_prefix}DynaarmSystem">
+          <command_interface name="freeze_mode" />
+        </gpio>
+      </xacro:if>
     </ros2_control>
   </xacro:macro>

File: urdf/dynaarm.urdf.xacro (robot description, xacro)
@@ -60,5 +60,6 @@
                                 drive_parameter_folder="${drive_parameter_folder_internal}"
                                 drive_parameter_folder_default="${default_drive_parameter_folder}"
-                                ethercat_addresses="${ethercat_addresses}"/>
+                                ethercat_addresses="${ethercat_addresses}"
+                                mode="${mode}"/>
   </xacro:macro>
   <!-- -->

File: urdf/dynaarm_standalone.urdf.xacro (robot description, xacro)
@@ -25,4 +25,5 @@
   <!-- Path to ros2_control controller config file -->
   <xacro:arg name="controller_path" default="" />
+  <xacro:arg name="namespace" default="" />
   <xacro:include filename="$(find dynaarm_description)/urdf/dynaarm.urdf.xacro" />
   <link name="base_link" />

Commit message: added duatic_ prefix

File: urdf/common/dynaarm.ros2control.xacro (robot description, xacro)
@@ -44,5 +44,5 @@
         </xacro:if>
         <xacro:if value="${mode == 'mock'}">
-          <plugin>dynaarm_driver/DynaarmMockHardwareInterface</plugin>
+          <plugin>duatic_dynaarm_driver/DynaarmMockHardwareInterface</plugin>
           <param name="tf_prefix">${tf_prefix}</param>
           <param name="start_in_freeze_mode">${start_in_freeze_mode}</param>
@@ -52,5 +52,5 @@
         </xacro:if>
         <xacro:if value="${mode == 'real'}">
-          <plugin>dynaarm_driver/DynaArmHardwareInterface</plugin>
+          <plugin>duatic_dynaarm_driver/DynaArmHardwareInterface</plugin>
           <param name="ethercat_bus">${ethercat_bus}</param>
           <param name="tf_prefix">${tf_prefix}</param>

File: urdf/common/dynaarm_common.urdf.xacro (robot description, xacro)
@@ -31,5 +31,5 @@
                 <geometry>
                     <mesh
-                        filename="file://$(find dynaarm_description)/meshes/${version}/${file_name}"
+                        filename="file://$(find duatic_dynaarm_description)/meshes/${version}/${file_name}"
                         scale="1.0 1.0 1.0" />
                 </geometry>
@@ -51,5 +51,5 @@
                 <geometry>
                     <mesh
-                        filename="file://$(find dynaarm_description)/meshes/${version}/${file_name}"
+                        filename="file://$(find duatic_dynaarm_description)/meshes/${version}/${file_name}"
                         scale="1.0 1.0 1.0" />
                 </geometry>
@@ -67,5 +67,5 @@
                 <geometry>
                     <mesh
-                        filename="file://$(find dynaarm_description)/meshes/${version}/${file_name}"
+                        filename="file://$(find duatic_dynaarm_description)/meshes/${version}/${file_name}"
                         scale="1.0 1.0 1.0" />
                 </geometry>

File: urdf/dynaarm.urdf.xacro (robot description, xacro)
@@ -28,10 +28,10 @@
     params="tf_prefix parent_link collision:='simple' dof mode ethercat_bus drive_order:='' start_in_freeze_mode:=false drive_parameter_folder:='' covers version *origin">
     <!-- Allow the user to pass the drive order file -->
-    <xacro:property name="default_drive_order_file" value="$(find dynaarm_description)/urdf/common/${version}/drive_order.yaml" />
+    <xacro:property name="default_drive_order_file" value="$(find duatic_dynaarm_description)/urdf/common/${version}/drive_order.yaml" />
     <xacro:property name="drive_order_file" value="${default_drive_order_file if drive_order == '' else drive_order}" />
     <!-- Obtain the EtherCAT drive order (address order list) -->
     <xacro:property name="ethercat_addresses" value="${xacro.load_yaml(drive_order_file)}"/>
     <!--Allow the user to pass a custom folder for drive parameters-->
-    <xacro:property name="default_drive_parameter_folder" value="$(find dynaarm_driver)/config/${version}" />
+    <xacro:property name="default_drive_parameter_folder" value="$(find duatic_dynaarm_driver)/config/${version}" />
     <xacro:if value="${drive_parameter_folder == ''}">
       <xacro:property name="drive_parameter_folder_internal" value="${default_drive_parameter_folder}" />
@@ -42,8 +42,8 @@
     <!-- Set ee_parent based on the specified DoF -->
     <xacro:property name="ee_parent" value="${base}" />
-    <xacro:include filename="$(find dynaarm_description)/urdf/common/dynaarm_common.urdf.xacro" />
+    <xacro:include filename="$(find duatic_dynaarm_description)/urdf/common/dynaarm_common.urdf.xacro" />
     <!-- Include the version specific information and also load the ethercat addresses from the drive file -->
-    <xacro:include filename="$(find dynaarm_description)/urdf/common/${version}/dynaarm_parameters.urdf.xacro" />
-    <xacro:include filename="$(find dynaarm_description)/urdf/common/dynaarm.ros2control.xacro" />
+    <xacro:include filename="$(find duatic_dynaarm_description)/urdf/common/${version}/dynaarm_parameters.urdf.xacro" />
+    <xacro:include filename="$(find duatic_dynaarm_description)/urdf/common/dynaarm.ros2control.xacro" />
     <xacro:dynaarm_joint_fixed joint_name="${joint_base_name}"
       parent="${parent_link}"

File: urdf/dynaarm_standalone.urdf.xacro (robot description, xacro)
@@ -25,5 +25,5 @@
   <!-- Path to ros2_control controller config file -->
   <xacro:arg name="controller_path" default="" />
-  <xacro:include filename="$(find dynaarm_description)/urdf/dynaarm.urdf.xacro" />
+  <xacro:include filename="$(find duatic_dynaarm_description)/urdf/dynaarm.urdf.xacro" />
   <link name="base_link" />
   <!-- create an instance of the dynaarm xacro macro and fix its base, move it up such that it doesn't intersect with the ground -->

File: urdf/dynaarm_standalone_dual.urdf.xacro (robot description, xacro)
@@ -24,5 +24,5 @@
   <!-- Path to ros2_control controller config file -->
   <xacro:arg name="controller_path" default="" />
-  <xacro:include filename="$(find dynaarm_description)/urdf/dynaarm.urdf.xacro" />
+  <xacro:include filename="$(find duatic_dynaarm_description)/urdf/dynaarm.urdf.xacro" />
   <link name="base_link" />
   <!-- create two dynaarms and fix their bases, move them up such that they do not intersect with the ground -->
@@ -50,5 +50,5 @@
   <!-- DynaArm Gazebo Ros2 Control-->
   <!-- Gazebo Ros2 Control -->
-  <xacro:include filename="$(find duatic_control)/urdf/plugins.urdf.xacro" />
+  <xacro:include filename="$(find duatic_duatic_control)/urdf/plugins.urdf.xacro" />
   <xacro:control namespace="$(arg namespace)">
     <remapping>cmd_vel:=cmd_vel</remapping> <!-- TODO: This line only exists, because otherwise the xacro doesn't compile -->

Commit message: move default drive configuration folder path resolution into ros2control xacro

File: urdf/common/dynaarm.ros2control.xacro (robot description, xacro)
@@ -62,5 +62,13 @@
     </joint>
   </xacro:macro>
-  <xacro:macro name="dynaarm_ros2_control" params="tf_prefix namespace:='' ethercat_bus start_in_freeze_mode drive_parameter_folder drive_parameter_folder_default ethercat_addresses mode">
+  <xacro:macro name="dynaarm_ros2_control" params="tf_prefix namespace:='' ethercat_bus start_in_freeze_mode drive_parameter_folder:='' ethercat_addresses mode">
+    <!--Allow the user to pass a custom folder for drive parameters-->
+    <xacro:property name="default_drive_parameter_folder" value="$(find duatic_dynaarm_driver)/config/${version}" />
+    <xacro:if value="${drive_parameter_folder == ''}">
+      <xacro:property name="drive_parameter_folder_internal" value="${default_drive_parameter_folder}" />
+    </xacro:if>
+    <xacro:unless value="${drive_parameter_folder == ''}">
+      <xacro:property name="drive_parameter_folder_internal" value="${drive_parameter_folder}" />
+    </xacro:unless>
     <ros2_control name="${tf_prefix}DynaarmSystem" type="system">
       <hardware>
@@ -79,6 +87,6 @@
           <param name="tf_prefix">${tf_prefix}</param>
           <param name="start_in_freeze_mode">${start_in_freeze_mode}</param>
-          <param name="drive_parameter_folder">${drive_parameter_folder}</param>
-          <param name="drive_parameter_folder_default">${drive_parameter_folder_default}</param>
+          <param name="drive_parameter_folder">${drive_parameter_folder_internal}</param>
+          <param name="drive_parameter_folder_default">${default_drive_parameter_folder}</param>
           <param name="initial_positions">[0.05, 0.05, 0.10, 0.05, 0.05, 0.05]</param>
         </xacro:if>
@@ -88,6 +96,6 @@
           <param name="tf_prefix">${tf_prefix}</param>
           <param name="start_in_freeze_mode">${start_in_freeze_mode}</param>
-          <param name="drive_parameter_folder">${drive_parameter_folder}</param>
-          <param name="drive_parameter_folder_default">${drive_parameter_folder_default}</param>
+          <param name="drive_parameter_folder">${drive_parameter_folder_internal}</param>
+          <param name="drive_parameter_folder_default">${default_drive_parameter_folder}</param>
         </xacro:if>
       </hardware>

File: urdf/dynaarm.urdf.xacro (robot description, xacro)
@@ -32,12 +32,4 @@
     <!-- Obtain the EtherCAT drive order (address order list) -->
     <xacro:property name="ethercat_addresses" value="${xacro.load_yaml(drive_order_file)}"/>
-    <!--Allow the user to pass a custom folder for drive parameters-->
-    <xacro:property name="default_drive_parameter_folder" value="$(find duatic_dynaarm_driver)/config/${version}" />
-    <xacro:if value="${drive_parameter_folder == ''}">
-      <xacro:property name="drive_parameter_folder_internal" value="${default_drive_parameter_folder}" />
-    </xacro:if>
-    <xacro:unless value="${drive_parameter_folder == ''}">
-      <xacro:property name="drive_parameter_folder_internal" value="${drive_parameter_folder}" />
-    </xacro:unless>
     <!-- Set ee_parent based on the specified DoF -->
     <xacro:property name="ee_parent" value="${base}" />
@@ -58,6 +50,5 @@
                                 ethercat_bus="${ethercat_bus}"
                                 start_in_freeze_mode="${start_in_freeze_mode}"
-                                drive_parameter_folder="${drive_parameter_folder_internal}"
-                                drive_parameter_folder_default="${default_drive_parameter_folder}"
+                                drive_parameter_folder="${drive_parameter_folder}"
                                 ethercat_addresses="${ethercat_addresses}"
                                 mode="${mode}"/>
