Commit message: reduce dynaarm.xacro and examples to the bare minimum

File: urdf/dynaarm.urdf.xacro (robot description, xacro)
@@ -26,10 +26,5 @@
   <!-- -->
   <xacro:macro name="dynaarm"
-    params="tf_prefix parent_link collision:='simple' dof mode ethercat_bus drive_order:='' start_in_freeze_mode:=false drive_parameter_folder:='' covers version *origin">
-    <!-- Allow the user to pass the drive order file -->
-    <xacro:property name="default_drive_order_file" value="$(find duatic_dynaarm_description)/urdf/common/${version}/drive_order.yaml" />
-    <xacro:property name="drive_order_file" value="${default_drive_order_file if drive_order == '' else drive_order}" />
-    <!-- Obtain the EtherCAT drive order (address order list) -->
-    <xacro:property name="ethercat_addresses" value="${xacro.load_yaml(drive_order_file)}"/>
+    params="tf_prefix parent_link collision:='simple' dof  covers version *origin">
     <!-- Set ee_parent based on the specified DoF -->
     <xacro:property name="ee_parent" value="${base}" />
@@ -37,5 +32,4 @@
     <!-- Include the version specific information and also load the ethercat addresses from the drive file -->
     <xacro:include filename="$(find duatic_dynaarm_description)/urdf/common/${version}/dynaarm_parameters.urdf.xacro" />
-    <xacro:include filename="$(find duatic_dynaarm_description)/urdf/common/dynaarm.ros2control.xacro" />
     <xacro:dynaarm_joint_fixed joint_name="${joint_base_name}"
       parent="${parent_link}"
@@ -46,11 +40,4 @@
     <xacro:dynaarm_main_body />
     <xacro:dynaarm_tool />
-    <!--ros2control-->
-    <xacro:dynaarm_ros2_control tf_prefix="${tf_prefix}"
-                                ethercat_bus="${ethercat_bus}"
-                                start_in_freeze_mode="${start_in_freeze_mode}"
-                                drive_parameter_folder="${drive_parameter_folder}"
-                                ethercat_addresses="${ethercat_addresses}"
-                                mode="${mode}"/>
   </xacro:macro>
   <!-- -->

File: urdf/dynaarm_standalone.urdf.xacro (robot description, xacro)
@@ -23,5 +23,4 @@
 <robot name="dynaarm" xmlns:xacro="http://www.ros.org/wiki/xacro">
   <!--Example single arm setup-->
-  <xacro:arg name="namespace" default="" />
   <xacro:arg name="tf_prefix" default="" />
   <!-- e.g.: 6-->
@@ -29,14 +28,8 @@
   <!-- collision: simple, complex -->
   <xacro:arg name="collision" default="simple" />
-  <!-- real, mock, sim -->
-  <xacro:arg name="mode" default="mock" />
-  <!-- physical ethercat bus, only used for real -->
-  <xacro:arg name="ethercat_bus" default="eth0" />
   <!-- Change to add covers to the arm -->
   <xacro:arg name="covers" default="false" />
   <!-- v1, v2, ... -->
   <xacro:arg name="version" default="baracuda12" />
-  <!-- Path to ros2_control controller config file -->
-  <xacro:arg name="controller_path" default="" />
   <xacro:include filename="$(find duatic_dynaarm_description)/urdf/dynaarm.urdf.xacro" />
   <link name="base_link" />
@@ -46,6 +39,4 @@
                 dof="$(arg dof)"
                 collision="$(arg collision)"
-                mode="$(arg mode)"
-                ethercat_bus="$(arg ethercat_bus)"
                 covers="$(arg covers)"
                 version="$(arg version)">

File: urdf/dynaarm_standalone_dual.urdf.xacro (robot description, xacro)
@@ -28,14 +28,8 @@
   <!-- collision: simple, complex-->
   <xacro:arg name="collision" default="complex" />
-  <!-- real, mock, sim -->
-  <xacro:arg name="mode" default="mock" />
-  <!-- physical ethercat bus, only used for real -->
-  <xacro:arg name="ethercat_bus" default="eth0" />
   <!-- Change to add covers to the arm -->
   <xacro:arg name="covers" default="false" />
   <!-- v1, v2, ... -->
   <xacro:arg name="version" default="baracuda12" />
-  <!-- Path to ros2_control controller config file -->
-  <xacro:arg name="controller_path" default="" />
   <xacro:include filename="$(find duatic_dynaarm_description)/urdf/dynaarm.urdf.xacro" />
   <link name="base_link" />
@@ -44,6 +38,4 @@
                 parent_link="base_link"
                 dof="$(arg dof)"
-                mode="$(arg mode)"
-                ethercat_bus="$(arg ethercat_bus)"
                 covers="$(arg covers)"
                 collision="$(arg collision)"
@@ -55,6 +47,4 @@
                 parent_link="base_link"
                 dof="$(arg dof)"
-                mode="$(arg mode)"
-                ethercat_bus="$(arg ethercat_bus)"
                 covers="$(arg covers)"
                 collision="$(arg collision)"

Commit message: Fix circular dependency (#63)
* move default drive configuration folder path resolution into ros2control xacro

* move gazebo import into ros2control xacro

* also remove it from standalone

* reduce dynaarm.xacro and examples to the bare minimum

* clear repos.list

* fix test launch

File: urdf/dynaarm.urdf.xacro (robot description, xacro)
@@ -26,18 +26,5 @@
   <!-- -->
   <xacro:macro name="dynaarm"
-    params="tf_prefix parent_link collision:='simple' dof mode ethercat_bus drive_order:='' start_in_freeze_mode:=false drive_parameter_folder:='' covers version *origin">
-    <!-- Allow the user to pass the drive order file -->
-    <xacro:property name="default_drive_order_file" value="$(find duatic_dynaarm_description)/urdf/common/${version}/drive_order.yaml" />
-    <xacro:property name="drive_order_file" value="${default_drive_order_file if drive_order == '' else drive_order}" />
-    <!-- Obtain the EtherCAT drive order (address order list) -->
-    <xacro:property name="ethercat_addresses" value="${xacro.load_yaml(drive_order_file)}"/>
-    <!--Allow the user to pass a custom folder for drive parameters-->
-    <xacro:property name="default_drive_parameter_folder" value="$(find duatic_dynaarm_driver)/config/${version}" />
-    <xacro:if value="${drive_parameter_folder == ''}">
-      <xacro:property name="drive_parameter_folder_internal" value="${default_drive_parameter_folder}" />
-    </xacro:if>
-    <xacro:unless value="${drive_parameter_folder == ''}">
-      <xacro:property name="drive_parameter_folder_internal" value="${drive_parameter_folder}" />
-    </xacro:unless>
+    params="tf_prefix parent_link collision:='simple' dof  covers version *origin">
     <!-- Set ee_parent based on the specified DoF -->
     <xacro:property name="ee_parent" value="${base}" />
@@ -45,5 +32,4 @@
     <!-- Include the version specific information and also load the ethercat addresses from the drive file -->
     <xacro:include filename="$(find duatic_dynaarm_description)/urdf/common/${version}/dynaarm_parameters.urdf.xacro" />
-    <xacro:include filename="$(find duatic_dynaarm_description)/urdf/common/dynaarm.ros2control.xacro" />
     <xacro:dynaarm_joint_fixed joint_name="${joint_base_name}"
       parent="${parent_link}"
@@ -54,12 +40,4 @@
     <xacro:dynaarm_main_body />
     <xacro:dynaarm_tool />
-    <!--ros2control-->
-    <xacro:dynaarm_ros2_control tf_prefix="${tf_prefix}"
-                                ethercat_bus="${ethercat_bus}"
-                                start_in_freeze_mode="${start_in_freeze_mode}"
-                                drive_parameter_folder="${drive_parameter_folder_internal}"
-                                drive_parameter_folder_default="${default_drive_parameter_folder}"
-                                ethercat_addresses="${ethercat_addresses}"
-                                mode="${mode}"/>
   </xacro:macro>
   <!-- -->

File: urdf/dynaarm_standalone.urdf.xacro (robot description, xacro)
@@ -23,5 +23,4 @@
 <robot name="dynaarm" xmlns:xacro="http://www.ros.org/wiki/xacro">
   <!--Example single arm setup-->
-  <xacro:arg name="namespace" default="" />
   <xacro:arg name="tf_prefix" default="" />
   <!-- e.g.: 6-->
@@ -29,31 +28,21 @@
   <!-- collision: simple, complex -->
   <xacro:arg name="collision" default="simple" />
-  <!-- real, mock, sim -->
-  <xacro:arg name="mode" default="mock" />
-  <!-- physical ethercat bus, only used for real -->
-  <xacro:arg name="ethercat_bus" default="eth0" />
   <!-- Change to add covers to the arm -->
   <xacro:arg name="covers" default="false" />
   <!-- v1, v2, ... -->
   <xacro:arg name="version" default="baracuda12" />
-  <!-- Path to ros2_control controller config file -->
-  <xacro:arg name="controller_path" default="" />
   <xacro:include filename="$(find duatic_dynaarm_description)/urdf/dynaarm.urdf.xacro" />
   <link name="base_link" />
   <!-- create an instance of the dynaarm xacro macro and fix its base, move it up such that it doesn't intersect with the ground -->
+  <!-- NOTE this is the bare minimum example of only the description
+    For an example on how to use ros2control with the dynaarm take a look at the duatic_dynaarm_demo repository
+  -->
   <xacro:dynaarm tf_prefix="$(arg tf_prefix)"
                 parent_link="base_link"
                 dof="$(arg dof)"
                 collision="$(arg collision)"
-                mode="$(arg mode)"
-                ethercat_bus="$(arg ethercat_bus)"
                 covers="$(arg covers)"
                 version="$(arg version)">
     <origin xyz="0 0 0" rpy="0.0 0.0 0.0" />
   </xacro:dynaarm>
-  <!-- Gazebo Ros2 Control -->
-  <xacro:include filename="$(find duatic_control)/urdf/plugins.urdf.xacro" />
-  <xacro:control namespace="$(arg namespace)">
-    <remapping>cmd_vel:=cmd_vel</remapping> <!-- TODO: This line only exists, because otherwise the xacro doesn't compile -->
-  </xacro:control>
 </robot>

File: urdf/dynaarm_standalone_dual.urdf.xacro (robot description, xacro)
@@ -28,14 +28,8 @@
   <!-- collision: simple, complex-->
   <xacro:arg name="collision" default="complex" />
-  <!-- real, mock, sim -->
-  <xacro:arg name="mode" default="mock" />
-  <!-- physical ethercat bus, only used for real -->
-  <xacro:arg name="ethercat_bus" default="eth0" />
   <!-- Change to add covers to the arm -->
   <xacro:arg name="covers" default="false" />
   <!-- v1, v2, ... -->
   <xacro:arg name="version" default="baracuda12" />
-  <!-- Path to ros2_control controller config file -->
-  <xacro:arg name="controller_path" default="" />
   <xacro:include filename="$(find duatic_dynaarm_description)/urdf/dynaarm.urdf.xacro" />
   <link name="base_link" />
@@ -44,6 +38,4 @@
                 parent_link="base_link"
                 dof="$(arg dof)"
-                mode="$(arg mode)"
-                ethercat_bus="$(arg ethercat_bus)"
                 covers="$(arg covers)"
                 collision="$(arg collision)"
@@ -55,6 +47,4 @@
                 parent_link="base_link"
                 dof="$(arg dof)"
-                mode="$(arg mode)"
-                ethercat_bus="$(arg ethercat_bus)"
                 covers="$(arg covers)"
                 collision="$(arg collision)"
@@ -62,9 +52,3 @@
     <origin xyz="1.0 0 0" rpy="0.0 0.0 0.0" />
   </xacro:dynaarm>
-  <!-- DynaArm Gazebo Ros2 Control-->
-  <!-- Gazebo Ros2 Control -->
-  <xacro:include filename="$(find duatic_duatic_control)/urdf/plugins.urdf.xacro" />
-  <xacro:control namespace="$(arg namespace)">
-    <remapping>cmd_vel:=cmd_vel</remapping> <!-- TODO: This line only exists, because otherwise the xacro doesn't compile -->
-  </xacro:control>
 </robot>

Commit message: rename dynaarm macro to dynaarm_description

File: urdf/dynaarm.urdf.xacro (robot description, xacro)
@@ -25,5 +25,5 @@
   <!-- DynaArm Macro-->
   <!-- -->
-  <xacro:macro name="dynaarm"
+  <xacro:macro name="dynaarm_description"
     params="tf_prefix parent_link collision:='simple' dof  covers version *origin">
     <!-- Set ee_parent based on the specified DoF -->

File: urdf/dynaarm_standalone.urdf.xacro (robot description, xacro)
@@ -38,5 +38,5 @@
     For an example on how to use ros2control with the dynaarm take a look at the duatic_dynaarm_demo repository
   -->
-  <xacro:dynaarm tf_prefix="$(arg tf_prefix)"
+  <xacro:dynaarm_description tf_prefix="$(arg tf_prefix)"
                 parent_link="base_link"
                 dof="$(arg dof)"
@@ -45,4 +45,4 @@
                 version="$(arg version)">
     <origin xyz="0 0 0" rpy="0.0 0.0 0.0" />
-  </xacro:dynaarm>
+  </xacro:dynaarm_description>
 </robot>

File: urdf/dynaarm_standalone_dual.urdf.xacro (robot description, xacro)
@@ -35,5 +35,5 @@
   <link name="base_link" />
   <!-- create two dynaarms and fix their bases, move them up such that they do not intersect with the ground -->
-  <xacro:dynaarm tf_prefix="$(arg tf_prefix)_1/"
+  <xacro:dynaarm_description tf_prefix="$(arg tf_prefix)_1/"
                 parent_link="base_link"
                 dof="$(arg dof)"
@@ -42,7 +42,7 @@
                 version="$(arg version)">
     <origin xyz="0 0 0" rpy="0.0 0.0 0.0" />
-  </xacro:dynaarm>
+  </xacro:dynaarm_description>
   <!-- Note: for a real world application you would pass different parameters for both arms (e.g. different ethercat_bus)-->
-  <xacro:dynaarm tf_prefix="$(arg tf_prefix)_2/"
+  <xacro:dynaarm_description tf_prefix="$(arg tf_prefix)_2/"
                 parent_link="base_link"
                 dof="$(arg dof)"
@@ -51,4 +51,4 @@
                 version="$(arg version)">
     <origin xyz="1.0 0 0" rpy="0.0 0.0 0.0" />
-  </xacro:dynaarm>
+  </xacro:dynaarm_description>
 </robot>
